File: documentation/diagrams/plant-helper kicad/plant-helper.kicad_sch (KiCad schematic)
At the start: 17 parts, among them U1 ESP32-S3-WROOM-2, U2 TLC555xP

Commit message: edit to kicad file
Parts:
- removed U1: ESP32-S3-WROOM-2, RF_Module:ESP32-S3-WROOM-2, symbol RF_Module:ESP32-S3-WROOM-2
- added C5: C, symbol Device:C
- added R8: R, symbol Device:R
- added U3: ESP32-WROOM-32D, RF_Module:ESP32-WROOM-32D, symbol RF_Module:ESP32-WROOM-32D
Connections:
- net GND: now also C5.1; no longer C4.2
- net at R6.1: now also U3.28 (IO17)
- net at R5.1: now also U3.27 (IO16)
- net at C1.2, D4.1 (K), R1.2: now also U3.7 (IO35)
- net at R7.1: now also U3.26 (IO4)
- new net: U3.1 (GND), U3.15 (GND), U3.38 (GND), U3.39 (GND)
- new net: C5.2, R8.1, U3.2 (VDD)
- new net: R8.2, U3.3 (EN)
Other:
- moved on the sheet: C1, C2, C3, C4, D1, D2, D3, D4, R1, R2, R3, R4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
